File: Azula Head Piece Light.sch (KiCad schematic (older format))
At the start: 11 parts, among them SW1 SW_DIP_x03

Commit message: Fix LED orientation and switch wiring
Fix LED orientation and switch wiring
Version 1.0.1
Parts:
- L1: Description (none) -> None; Manufacturer Name (none) -> None; Manufacturer Part No. (none) -> None; Source (none) -> None
Connections:
- net labels added: BAT+
- net labels removed: BATSWITCH
- wire segments 34 -> 42
Other:
- moved on the sheet: D1, D2, D3
Changed lines of the file:
@@
 F 8 "LED Lighting J White, Neutral 4000K 3-Step MacAdam Ellipse 2.71V 65mA 120° 2212 (5630 Metric)" H 6850 4100 50  0001 C CNN "Description"
 	1    6850 4100
-	0    -1   -1   0
+	0    1    1    0
 $EndComp
 $Comp
@@
 Connection ~ 6400 3450
 Wire Wire Line
-	6400 3450 6650 3450
+	6400 3450 6600 3450
 Wire Wire Line
 	5950 3550 5950 3450
@@
 F 8 "LED Lighting J White, Neutral 4000K 3-Step MacAdam Ellipse 2.71V 65mA 120° 2212 (5630 Metric)" H 6400 4100 50  0001 C CNN "Description"
 	1    6400 4100
-	0    -1   -1   0
+	0    1    1    0
 $EndComp
 $Comp
@@
 F 8 "LED Lighting J White, Neutral 4000K 3-Step MacAdam Ellipse 2.71V 65mA 120° 2212 (5630 Metric)" H 5950 4100 50  0001 C CNN "Description"
 	1    5950 4100
-	0    -1   -1   0
+	0    1    1    0
 $EndComp
 $Comp
@@
 L Azula~Head~Piece:SW_DIP_x03 SW1
 U 1 1 5F182016
-P 5550 3350
-F 0 "SW1" H 5550 3083 50  0000 C CNN
-F 1 "SW_DIP_x03" H 5550 3174 50  0000 C CNN
-F 2 "Azula Head Piece Light:CL-SB-22A_HandSolder_Edge" H 5550 3350 50  0001 C CNN
-F 3 "https://www.nidec-copal-electronics.com/e/catalog/switch/cl-sb.pdf" H 5550 3350 50  0001 C CNN
-F 4 "Slide Switch DPDT Surface Mount, Right Angle" H 5550 3350 50  0001 C CNN "Description"
-F 5 "Nidec Copal Electronics" H 5550 3350 50  0001 C CNN "Manufacturer Name"
-F 6 "CL-SB-22A-11T" H 5550 3350 50  0001 C CNN "Manufacturer Part No."
-F 7 "Digikey" H 5550 3350 50  0001 C CNN "Source"
-F 8 "563-1340-1-ND" H 5550 3350 50  0001 C CNN "Source Part No."
-	1    5550 3350
-	-1   0    0    1
-$EndComp
-Wire Wire Line
-	5800 3450 5850 3450
+P 5600 3450
+F 0 "SW1" V 6000 3550 50  0000 C CNN
+F 1 "SW_DIP_x03" V 6100 3550 50  0000 C CNN
+F 2 "Azula Head Piece Light:CL-SB-22A_HandSolder_Edge" H 5600 3450 50  0001 C CNN
+F 3 "https://www.nidec-copal-electronics.com/e/catalog/switch/cl-sb.pdf" H 5600 3450 50  0001 C CNN
+F 4 "Slide Switch DPDT Surface Mount, Right Angle" H 5600 3450 50  0001 C CNN "Description"
+F 5 "Nidec Copal Electronics" H 5600 3450 50  0001 C CNN "Manufacturer Name"
+F 6 "CL-SB-22A-11T" H 5600 3450 50  0001 C CNN "Manufacturer Part No."
+F 7 "Digikey" H 5600 3450 50  0001 C CNN "Source"
+F 8 "563-1340-1-ND" H 5600 3450 50  0001 C CNN "Source Part No."
+	1    5600 3450
+	0    -1   -1   0
+$EndComp
 Connection ~ 4750 4350
-Wire Wire Line
-	5800 3350 5850 3350
-Wire Wire Line
-	5850 3350 5850 3450
-Connection ~ 5850 3450
-Wire Wire Line
-	5850 3450 5950 3450
-Wire Wire Line
-	5300 3350 5250 3350
-Wire Wire Line
-	5250 3350 5250 3450
-Connection ~ 5250 3450
-Wire Wire Line
-	5250 3450 5300 3450
-NoConn ~ 5800 3550
-NoConn ~ 5300 3550
+NoConn ~ 5400 3700
+NoConn ~ 5400 3200
 Wire Wire Line
 	6850 3450 6950 3450
@@
 NoConn ~ 4700 3600
 Text Label 4800 3450 0    50   ~ 0
-BATSWITCH
-Wire Wire Line
-	4800 3450 5250 3450
+BAT+
 Wire Wire Line
 	4750 4350 5100 4350
@@
 L Frequently_Used_LE:PWR_FLAG #FLG0101
 U 1 1 5F5939B4
-P 6650 3450
-F 0 "#FLG0101" H 6650 3525 50  0001 C CNN
-F 1 "PWR_FLAG" H 6650 3623 50  0000 C CNN
-F 2 "" H 6650 3450 50  0001 C CNN
-F 3 "~" H 6650 3450 50  0001 C CNN
-	1    6650 3450
-	1    0    0    -1
-$EndComp
-Connection ~ 6650 3450
-Wire Wire Line
-	6650 3450 6850 3450
+P 6600 3350
+F 0 "#FLG0101" H 6600 3425 50  0001 C CNN
+F 1 "PWR_FLAG" H 6600 3523 50  0000 C CNN
+F 2 "" H 6600 3350 50  0001 C CNN
+F 3 "~" H 6600 3350 50  0001 C CNN
+	1    6600 3350
+	1    0    0    -1
+$EndComp
+Connection ~ 6600 3450
+Wire Wire Line
+	6600 3450 6850 3450
 $Comp
 L Frequently_Used_LE:PWR_FLAG #FLG0102
 U 1 1 5F595814
-P 5300 4350
-F 0 "#FLG0102" H 5300 4425 50  0001 C CNN
-F 1 "PWR_FLAG" H 5300 4523 50  0000 C CNN
-F 2 "" H 5300 4350 50  0001 C CNN
-F 3 "~" H 5300 4350 50  0001 C CNN
-	1    5300 4350
+P 5300 4250
+F 0 "#FLG0102" H 5300 4325 50  0001 C CNN
+F 1 "PWR_FLAG" H 5300 4423 50  0000 C CNN
+F 2 "" H 5300 4250 50  0001 C CNN
+F 3 "~" H 5300 4250 50  0001 C CNN
+	1    5300 4250
 	1    0    0    -1
 $EndComp
@@
 F 1 "Logo" H 7185 6205 50  0000 L CNN
 F 2 "Logos_LE:OSHW-Symbol_4mm_Silkscreen" H 7100 6250 50  0001 C CNN
-F 3 "" H 7100 6250 50  0001 C CNN
+F 3 "None" H 7100 6250 50  0001 C CNN
+F 4 "None" H 7100 6250 50  0001 C CNN "Description"
+F 5 "None" H 7100 6250 50  0001 C CNN "Manufacturer Name"
+F 6 "None" H 7100 6250 50  0001 C CNN "Manufacturer Part No."
+F 7 "None" H 7100 6250 50  0001 C CNN "Source"
 	1    7100 6250
 	1    0    0    -1
 $EndComp
+Wire Wire Line
+	5800 3450 5950 3450
+Wire Wire Line
+	4800 3450 5200 3450
+Wire Wire Line
+	5500 3200 5500 3100
+Wire Wire Line
+	5200 3100 5200 3450
+Wire Wire Line
+	5200 3450 5200 3800
+Wire Wire Line
+	5500 3800 5500 3700
+Wire Wire Line
+	5600 3700 5600 3800
+Wire Wire Line
+	5600 3800 5800 3800
+Wire Wire Line
+	5800 3800 5800 3450
+Connection ~ 5200 3450
+Wire Wire Line
+	5200 3100 5500 3100
+Wire Wire Line
+	5200 3800 5500 3800
+Wire Wire Line
+	5600 3200 5600 3100
+Wire Wire Line
+	5600 3100 5800 3100
+Wire Wire Line
+	5800 3100 5800 3450
+Connection ~ 5800 3450
+Wire Wire Line
+	6600 3350 6600 3450
+Wire Wire Line
+	5300 4250 5300 4350
 $EndSCHEMATC

Commit message: Fixed pin out on LED
Fixed pin out on LED
Other:
- moved on the sheet: D1, D2, D3
Changed lines of the file:
@@
 F 8 "LED Lighting J White, Neutral 4000K 3-Step MacAdam Ellipse 2.71V 65mA 120° 2212 (5630 Metric)" H 6850 4100 50  0001 C CNN "Description"
 	1    6850 4100
-	0    1    1    0
+	0    -1   -1   0
 $EndComp
 $Comp
@@
 F 8 "LED Lighting J White, Neutral 4000K 3-Step MacAdam Ellipse 2.71V 65mA 120° 2212 (5630 Metric)" H 6400 4100 50  0001 C CNN "Description"
 	1    6400 4100
-	0    1    1    0
+	0    -1   -1   0
 $EndComp
 $Comp
@@
 F 8 "LED Lighting J White, Neutral 4000K 3-Step MacAdam Ellipse 2.71V 65mA 120° 2212 (5630 Metric)" H 5950 4100 50  0001 C CNN "Description"
 	1    5950 4100
-	0    1    1    0
+	0    -1   -1   0
 $EndComp
 $Comp

Commit message: Added fiducials
Parts:
- added FID1, FID2, FID3: Fiducial, Fiducial_LE:Fiducial_1mm_Mask2mm, symbol Mechanical_LE:Fiducial
Other:
- note added: "Additional Features"
- note added: "Schematic"
- moved on the sheet: L1
Changed lines of the file:
@@
 L Frequently_Used_LE:Logo L1
 U 1 1 5F598CE9
-P 7100 6250
-F 0 "L1" H 7185 6296 50  0000 L CNN
-F 1 "Logo" H 7185 6205 50  0000 L CNN
-F 2 "Logos_LE:OSHW-Symbol_4mm_Silkscreen" H 7100 6250 50  0001 C CNN
-F 3 "None" H 7100 6250 50  0001 C CNN
-F 4 "None" H 7100 6250 50  0001 C CNN "Description"
-F 5 "None" H 7100 6250 50  0001 C CNN "Manufacturer Name"
-F 6 "None" H 7100 6250 50  0001 C CNN "Manufacturer Part No."
-F 7 "None" H 7100 6250 50  0001 C CNN "Source"
-	1    7100 6250
+P 8200 6150
+F 0 "L1" H 8285 6196 50  0000 L CNN
+F 1 "Logo" H 8285 6105 50  0000 L CNN
+F 2 "Logos_LE:OSHW-Symbol_4mm_Silkscreen" H 8200 6150 50  0001 C CNN
+F 3 "None" H 8200 6150 50  0001 C CNN
+F 4 "None" H 8200 6150 50  0001 C CNN "Description"
+F 5 "None" H 8200 6150 50  0001 C CNN "Manufacturer Name"
+F 6 "None" H 8200 6150 50  0001 C CNN "Manufacturer Part No."
+F 7 "None" H 8200 6150 50  0001 C CNN "Source"
+	1    8200 6150
 	1    0    0    -1
 $EndComp
@@
 Wire Wire Line
 	5300 4250 5300 4350
+$Comp
+L Mechanical_LE:Fiducial FID1
+U 1 1 5F687C5C
+P 8750 6150
+F 0 "FID1" H 8835 6196 50  0000 L CNN
+F 1 "Fiducial" H 8750 5800 50  0001 C CNN
+F 2 "Fiducial_LE:Fiducial_1mm_Mask2mm" H 8750 6000 50  0001 C CNN
+F 3 "None" H 8700 6150 50  0001 C CNN
+F 4 "TOP1" H 8835 6105 50  0000 L CNN "Name"
+F 5 "None" H 8750 5700 50  0001 C CNN "Manufacturer Name"
+F 6 "None" H 8750 5600 50  0001 C CNN "Manufacturer Part No."
+F 7 "None" H 8750 5400 50  0001 C CNN "Source"
+F 8 "None" H 8750 5500 50  0001 C CNN "Source Part No."
+F 9 "Fiducial mark" H 8750 5900 50  0001 C CNN "Description"
+	1    8750 6150
+	1    0    0    -1
+$EndComp
+$Comp
+L Mechanical_LE:Fiducial FID2
+U 1 1 5F689A36
+P 9300 6150
+F 0 "FID2" H 9385 6196 50  0000 L CNN
+F 1 "Fiducial" H 9300 5800 50  0001 C CNN
+F 2 "Fiducial_LE:Fiducial_1mm_Mask2mm" H 9300 6000 50  0001 C CNN
+F 3 "None" H 9250 6150 50  0001 C CNN
+F 4 "TOP2" H 9385 6105 50  0000 L CNN "Name"
+F 5 "None" H 9300 5700 50  0001 C CNN "Manufacturer Name"
+F 6 "None" H 9300 5600 50  0001 C CNN "Manufacturer Part No."
+F 7 "None" H 9300 5400 50  0001 C CNN "Source"
+F 8 "None" H 9300 5500 50  0001 C CNN "Source Part No."
+F 9 "Fiducial mark" H 9300 5900 50  0001 C CNN "Description"
+	1    9300 6150
+	1    0    0    -1
+$EndComp
+$Comp
+L Mechanical_LE:Fiducial FID3
+U 1 1 5F68A5FE
+P 9800 6150
+F 0 "FID3" H 9885 6196 50  0000 L CNN
+F 1 "Fiducial" H 9800 5800 50  0001 C CNN
+F 2 "Fiducial_LE:Fiducial_1mm_Mask2mm" H 9800 6000 50  0001 C CNN
+F 3 "None" H 9750 6150 50  0001 C CNN
+F 4 "TOP3" H 9885 6105 50  0000 L CNN "Name"
+F 5 "None" H 9800 5700 50  0001 C CNN "Manufacturer Name"
+F 6 "None" H 9800 5600 50  0001 C CNN "Manufacturer Part No."
+F 7 "None" H 9800 5400 50  0001 C CNN "Source"
+F 8 "None" H 9800 5500 50  0001 C CNN "Source Part No."
+F 9 "Fiducial mark" H 9800 5900 50  0001 C CNN "Description"
+	1    9800 6150
+	1    0    0    -1
+$EndComp
+Text Notes 8550 6450 0    79   ~ 16
+Additional Features
+Text Notes 5400 5000 0    79   ~ 16
+Schematic
 $EndSCHEMATC
